File: dev style rev0.1.brd (EAGLE design)
At the start: 50 x 50 mm, 55 parts, among them IC2 MCP73871, SW1 BUTTON-TL3330AF130QG, U1 PIC24FJ128GB204, U2 TELIT_RE866, U3 24LC32A-SOT23-5, U4 TITAN-X1-GMS-3302, U5 AT45DB161E-SHD2B-T, U6 LSM6DSL, U7 PAM2305AAB330, Y1 16MHz

Commit message: updated cell dev
Parts:
- moved SJ3 0.51 mm to (2.00, 25.0)
- renumbered IC2 to U8
Routing:
- net TELIT_RESET: track 32.8 -> 33.3 mm
Other:
- outline, holes or cut-outs redrawn
