File: cell version/dev style cell rev0.1.sch (EAGLE design)
At the start: 55 parts, among them IC2 MCP73871, SW1 BUTTON-TL3330AF130QG, U1 PIC24FJ128GB204, U2 TELIT_RE866, U3 24LC32A-SOT23-5, U4 TITAN-X1-GMS-3302, U5 AT45DB161E-SHD2B-T, U6 LSM6DSL, U7 PAM2305AAB330, Y1 16MHz

Commit message: updated cell dev
Parts:
- removed U2: TELIT_RE866, clackboard_lib:TELIT_RE866
- added CON1: SIMCARD_HOLDER_693022010811, clackboard_lib:SIMCARD_HOLDER_693022010811
- added J1: (no value), SparkFun-Connectors:USB_MICRO-B_SMT
- added LED3, LED4: GREEN, adafruit:LEDCHIP-LED0603
- added R13: 10K, resistor:R-US_R0402
- added R14, R15: 1K, resistor:R-US_R0402
- added TP1, TP2, TP3: PTR1PAD1-17, testpad:PTR1PAD1-17
- added U9: SIM7000A, clackboard_lib:SIM7000A
- renumbered IC2 to U8
Connections:
- new net N$21: U9.RF_ANT
- new net N$22: R13.1, SJ6.2, U9.PWRKEY
- new net N$23: CON1.C1, U9.SIM_VDD
- new net N$25: CON1.C3, U9.SIM_CLK
- new net N$26: CON1.C7, U9.SIM_DATA
- new net N$27: CON1.C2, U9.SIM_RST
- new net N$28: LED3.A, R14.1
- new net N$29: TP1.TP, U9.MDM_LOG_TX
- new net N$30: LED4.A, R15.1
- new net N$31: R15.2, U9.STATUS
- new net N$32: TP2.TP, U9.BOOT_CFG
- new net N$33: J1.VBUS, U9.USB_VBUS
- new net N$34: U9.GNSS_ANT
- new net N$36: TP3.TP, U9.VDD_EXT
- new net SIM_N: J1.D-, U9.USB_DM
- new net SIM_P: J1.D+, U9.USB_DP
- net 3.3V: now also R13.2; no longer U2.VDD_NRF_LORA@E1, U2.VDD_NRF_LORA@E2
- net GND: now also CON1.C5, CON1.PAD1, CON1.PAD2, J1.GND, J1.SHIELD, LED3.C, LED4.C, U9.GND@17, U9.GND@18, U9.GND@2, U9.GND@29, U9.GND@39, U9.GND@45, U9.GND@46, U9.GND@48, U9.GND@54, U9.GND@59, U9.GND@61, U9.GND@62, U9.GND@63, U9.GND@64, U9.GND@65; no longer U2.GND@C3, U2.GND@D1, U2.GND@D2, U2.GND@E3, U2.GND@F1, U2.GND@F2, U2.GND@F3, U2.GND@F6, U2.GND@G1, U2.GND@G3
- net IUR_IN: no longer U2.IUR-IN#
- net IUR_OUT: no longer U2.IUR-OUT#
- net N$11: no longer U2.TESTMODE
- net N$12: now also SJ3.1, U9.NRESET; no longer SJ6.2, U2.BOOT0
- net N$18: now also R14.2, U9.NETLIGHT; no longer SJ3.1, U2.RESET
- net PIC_CTS: now also U9.RTS; no longer U2.UART-RTS#
- net PIC_RTS: now also U9.CTS; no longer U2.UART-CTS#
- net PIC_RX: now also U9.TXD; no longer U2.UART-TXD
- net PIC_TX: now also U9.RXD; no longer U2.UART-RXD
- net VBAT: now also U9.VBAT@55, U9.VBAT@56, U9.VBAT@57
Other:
- note added: "SIM7000A Module"
- note removed: "LoRa Module"
- moved on the sheet: C11, C13, L2, R12, SJ3, SJ6, SJ7, SW1, U7

Commit message: added antennas and fiducials, finished routing, cleaned silk, added custom silk
Parts:
- added LED5: GREEN, adafruit:LEDCHIP-LED0603
- added R16: 1K, resistor:R-US_R0402
- added U$1, U$2, U$3, U$4: FIDUCIAL, adafruit:FIDUCIAL
- added X1, X2: (no value), adafruit:ANTENNA_U.FL
- renumbered SV1 to ICD3_HEADER
Connections:
- new net N$35: LED5.C, R16.2
- net 3.3V: now also LED5.A
- net GND: now also R16.1, X1.GND@0, X1.GND@1, X2.GND@0, X2.GND@1
- net N$21: now also X1.SIGNAL
- net N$34: now also X2.SIGNAL
Other:
- note added: "2.0"
- note added: "3V3"
- note added: "3V7-4V2"
- note added: "5V"
- note added: "CELL"
- note added: "FLASH"
- note added: "GPIO"
- note added: "GPS"
- note added: "I2C"
- note added: "MOTION SENSOR"
- note added: "PMU"
- note added: "SPI"
- note added: "STEP DOWN"
- note added: "UART0"
- note added: "UART1"
- note added: "USB"
- note added: "VBAT"
- note added: "VUSB"

Commit message: pushed after a while
Parts:
- removed U9: SIM7000A, clackboard_lib:SIM7000A
- added U2: TELIT_LE866, clackboard_lib:TELIT_LE866
Connections:
- removed net IUR_IN: U1.RP23/PMA0/PMALL/CN17/RC7
- removed net IUR_OUT: U1.AN7/C1INC/REFO/RP13/CTPLS/PMRD/CN13/RB13
- removed net N$29: TP1.TP, U9.MDM_LOG_TX
- removed net N$32: TP2.TP, U9.BOOT_CFG
- removed net N$33: J1.VBUS, U9.USB_VBUS
- removed net N$34: U9.GNSS_ANT, X2.SIGNAL
- new net DIV_ANT: U2.DIV_ANT
- new net MAIN_ANT: U2.MAIN_ANT, X2.SIGNAL
- new net N$42: SJ3.1
- new net N$47: TP1.TP
- new net N$48: TP2.TP
- new net VBUS: J1.VBUS
- net GND: now also U2.GND; no longer U9.GND@17, U9.GND@18, U9.GND@2, U9.GND@29, U9.GND@39, U9.GND@45, U9.GND@46, U9.GND@48, U9.GND@54, U9.GND@59, U9.GND@61, U9.GND@62, U9.GND@63, U9.GND@64, U9.GND@65
- net N$12: now also U2.VBATT, U2.VBATT_PA; no longer SJ3.1, U9.NRESET
- net N$18: no longer U9.NETLIGHT
- net N$21: no longer U9.RF_ANT
- net N$22: no longer U9.PWRKEY
- net N$23: now also U2.SIMVCC; no longer U9.SIM_VDD
- net N$25: now also CON1.C2, U2.SIMRST; no longer CON1.C3, U9.SIM_CLK
- net N$26: now also CON1.C3, U2.SIMCLK; no longer CON1.C7, U9.SIM_DATA
- net N$27: now also CON1.C7, U2.SIMIO; no longer CON1.C2, U9.SIM_RST
- net N$31: no longer U9.STATUS
- net N$36: no longer U9.VDD_EXT
- net PIC_CTS: now also U2.C105/RTS; no longer U9.RTS
- net PIC_RTS: now also U2.C106/CTS; no longer U9.CTS
- net PIC_RX: now also U2.TX/AUX; no longer U9.TXD
- net PIC_TX: now also U2.RX_AUX; no longer U9.RXD
- net SIM_N: now also U2.USB_D-; no longer U9.USB_DM
- net SIM_P: now also U2.USB_D+; no longer U9.USB_DP
- net VBAT: no longer U9.VBAT@55, U9.VBAT@56, U9.VBAT@57
Other:
- note added: "Telit_LE866 Module"
- note added: "thicc traces"
- note removed: "SIM7000A Module"
- moved on the sheet: CON1, J1, LED3, LED4, R13, R14, R15, SJ3, SJ6, SJ7, TP1, TP2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
