File: cell version/dev style sim7000a cell rev0.1.sch (EAGLE design)
At the start: 67 parts, among them CON1 SIMCARD_HOLDER_693022010811, SW1 BUTTON-TL3330AF130QG, U1 PIC24FJ128GB204, U3 24LC32A-SOT23-5, U4 TITAN-X1-GMS-3302, U5 AT45DB161E-SHD2B-T, U6 LSM6DSL, U7 PAM2305AAB330, U8 MCP73871, U9 SIM7000A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

Commit message: pushed after a while
Parts:
- added U$1, U$2, U$3, U$4: FIDUCIAL, adafruit:FIDUCIAL
- added X1, X2: (no value), adafruit:ANTENNA_U.FL
Connections:
- net GND: now also X1.GND@0, X1.GND@1, X2.GND@0, X2.GND@1
- net N$21: now also X1.SIGNAL
- net N$34: now also X2.SIGNAL
Changed lines of the file:
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@@
 <setting verticaltext="up"/>
 </settings>
-<grid distance="0.05" unitdist="inch" unit="inch" style="lines" multiple="1" display="no" altdistance="0.01" altunitdist="inch" altunit="inch"/>
+<grid distance="0.1" unitdist="inch" unit="inch" style="lines" multiple="1" display="no" altdistance="0.01" altunitdist="inch" altunit="inch"/>
 <layers>
 <layer number="1" name="Top" color="4" fill="1" visible="no" active="no"/>
@@
 <part name="SUPPLY23" library="SparkFun-PowerSymbols" deviceset="3.3V" device=""/>
 <part name="GND8" library="SparkFun-PowerSymbols" deviceset="GND" device=""/>
+<part name="X1" library="adafruit" library_urn="urn:adsk.eagle:library:420" deviceset="ANTENNA_U.FL" device=""/>
+<part name="GND41" library="SparkFun-PowerSymbols" deviceset="GND" device=""/>
+<part name="X2" library="adafruit" library_urn="urn:adsk.eagle:library:420" deviceset="ANTENNA_U.FL" device=""/>
+<part name="GND42" library="SparkFun-PowerSymbols" deviceset="GND" device=""/>
+<part name="U$1" library="adafruit" library_urn="urn:adsk.eagle:library:420" deviceset="FIDUCIAL" device=""/>
+<part name="U$2" library="adafruit" library_urn="urn:adsk.eagle:library:420" deviceset="FIDUCIAL" device=""/>
+<part name="U$3" library="adafruit" library_urn="urn:adsk.eagle:library:420" deviceset="FIDUCIAL" device=""/>
+<part name="U$4" library="adafruit" library_urn="urn:adsk.eagle:library:420" deviceset="FIDUCIAL" device=""/>
 </parts>
 <sheets>
@@
 <instance part="GND40" gate="1" x="195.58" y="200.66"/>
 <instance part="TP3" gate="G$1" x="213.36" y="231.14" rot="R270"/>
+<instance part="X1" gate="G$1" x="303.53" y="246.38" rot="MR0"/>
+<instance part="GND41" gate="1" x="308.61" y="234.95"/>
+<instance part="X2" gate="G$1" x="303.53" y="228.6" rot="MR0"/>
+<instance part="GND42" gate="1" x="307.34" y="217.17"/>
+<instance part="U$1" gate="G$1" x="411.48" y="81.28"/>
+<instance part="U$2" gate="G$1" x="411.48" y="73.66"/>
+<instance part="U$3" gate="G$1" x="411.48" y="66.04"/>
+<instance part="U$4" gate="G$1" x="411.48" y="58.42"/>
 </instances>
 <busses>
@@
 <pinref part="GND40" gate="1" pin="GND"/>
 </segment>
+<segment>
+<pinref part="X1" gate="G$1" pin="GND@0"/>
+<wire x1="306.07" y1="241.3" x2="308.61" y2="241.3" width="0.1524" layer="91"/>
+<wire x1="308.61" y1="241.3" x2="308.61" y2="238.76" width="0.1524" layer="91"/>
+<pinref part="X1" gate="G$1" pin="GND@1"/>
+<wire x1="308.61" y1="238.76" x2="308.61" y2="237.49" width="0.1524" layer="91"/>
+<wire x1="306.07" y1="238.76" x2="308.61" y2="238.76" width="0.1524" layer="91"/>
+<junction x="308.61" y="238.76"/>
+<pinref part="GND41" gate="1" pin="GND"/>
+</segment>
+<segment>
+<pinref part="X2" gate="G$1" pin="GND@0"/>
+<wire x1="306.07" y1="223.52" x2="307.34" y2="223.52" width="0.1524" layer="91"/>
+<wire x1="307.34" y1="223.52" x2="307.34" y2="220.98" width="0.1524" layer="91"/>
+<pinref part="X2" gate="G$1" pin="GND@1"/>
+<wire x1="307.34" y1="220.98" x2="307.34" y2="219.71" width="0.1524" layer="91"/>
+<wire x1="306.07" y1="220.98" x2="307.34" y2="220.98" width="0.1524" layer="91"/>
+<junction x="307.34" y="220.98"/>
+<pinref part="GND42" gate="1" pin="GND"/>
+</segment>
 </net>
 <net name="USB_N" class="0">
@@
 <segment>
 <pinref part="U9" gate="G$1" pin="RF_ANT"/>
-<wire x1="269.24" y1="246.38" x2="320.04" y2="246.38" width="0.1524" layer="91"/>
+<wire x1="269.24" y1="246.38" x2="298.45" y2="246.38" width="0.1524" layer="91"/>
+<pinref part="X1" gate="G$1" pin="SIGNAL"/>
 </segment>
 </net>
@@
 <segment>
 <pinref part="U9" gate="G$1" pin="GNSS_ANT"/>
-<wire x1="269.24" y1="228.6" x2="320.04" y2="228.6" width="0.1524" layer="91"/>
-</segment>
-</net>
+<wire x1="269.24" y1="228.6" x2="298.45" y2="228.6" width="0.1524" layer="91"/>
+<pinref part="X2" gate="G$1" pin="SIGNAL"/>
+</segment>
+</net>
